File: PCB/101 PCB/101 PCB.kicad_sch (KiCad schematic)
At the start: 56 parts, among them IC101 TPS563202DRLR, IC103 TPS563202DRLR, IC104 DRV8837DSGR, IC105 DRV8837DSGR, J1 TYPE-C-31-M-12, J102 Screw_Terminal_01x02, J103 Screw_Terminal_01x02, J104 Conn_01x04, J105 Conn_01x04, J106 Conn_01x04, J107 Conn_01x04, J108 Conn_01x04, J109 Conn_01x04, J110 Screw_Terminal_01x02, J111 SM04B-SRSS-TB(LF)(SN), U1 USBLC6-4SC6-ES, U101 ESP32-WROOM-32, U104 LSM6DS3, U106 STM32G431CBUx

Commit message: Board layout done
Parts:
- removed R5, R6: 5k1, Resistor_SMD:R_0402_1005Metric, symbol Device:R_Small
- added C119: 47u, Capacitor_SMD:CP_Elec_6.3x5.8, symbol Device:C_Polarized_Small
- added C120, C121, C122, C123, C126, C20: 100n, Capacitor_SMD:C_0402_1005Metric, symbol Device:C_Small
- added C124: 4u7, Capacitor_SMD:C_0402_1005Metric, symbol Device:C_Small
- added C125, C127: 1u, Capacitor_SMD:C_0402_1005Metric, symbol Device:C_Small
- added D104: ZMM10V, Diode_SMD:D_MiniMELF, symbol Diode:ZMMxx
- added J301: TC2030, Connector:Tag-Connect_TC2030-IDC-FP_2x03_P1.27mm_Vertical, symbol Connector:Conn_ARM_SWD_TagConnect_TC2030
- added Q101: DMP3028LFDE, 101 Footprints:DMP2066UFDE7, symbol DMP3028LFDE-7:DMP3028LFDE
- added R108, R113, R114: 330R, Resistor_SMD:R_0402_1005Metric, symbol Device:R_Small
- added R23: 10k, Resistor_SMD:R_0402_1005Metric, symbol Device:R_Small
- added S301 (x2): TS20-42-25-WT-160-SMT-TR, MSL Footprints:TS204225WT160SMTTRMSL, symbol TS20-42-25-WT-160-SMT-TR-MSL:TS20-42-25-WT-160-SMT-TR
- L101, L102: footprint (none) -> Inductor_SMD:L_Chilisin_BMRA00040420
- R101, R103, R104, R106: footprint (none) -> Resistor_SMD:R_0402_1005Metric
- R19: value 3k3 -> 1k
- R22: value 10k -> 1k
Connections:
- net BATT/4 is gone; now on net BATT/11: R19.1, R20.2, U101.4 (SENSOR_VP)
- net VBUS/2 is gone; now on net VBUS/11: R21.2, R22.1, U101.5 (SENSOR_VN)
- net +3.3V: now also U106.1 (VBAT), U106.21 (VDDA), U106.23 (VDD), U106.35 (VDD), U106.48 (VDD), C120.1, C121.1, C122.1, C123.1, C124.1, C125.1
- net +3V3: now also J301.1 (VCC), R23.2
- net +BATT: now also C119.1, D104.1 (K), Q101.4 (S_1), Q101.7 (S_2); no longer J110.1 (Pin_1)
- net CC1: now also U1.3 (IO2), U106.44 (PB6); no longer U1.1 (IO1)
- net CC2: now also U1.1 (IO1), U106.42 (PB4); no longer U1.3 (IO2)
- net EN: now also C20.1, R114.2, R23.1, S301.2 (NO_2)
- net ESP32_RX: now also U106.10 (PA2)
- net ESP32_TX: now also U106.11 (PA3)
- net GND: now also U106.49 (VSS), C119.2, C120.2, C121.2, C122.2, C123.2, C124.2, C125.2, C126.2, C127.2, C20.2, J301.5 (GND), R108.2, S301.3 (COM_1), S301.3 (COM_1)
- net GPIO12: now also A101.20 (D5)
- net GPIO13: now also A101.21 (D6)
- net GPIO14: now also A101.22 (D7)
- net GPIO15: now also A101.14 (SCL/A5)
- net GPIO16: now also A101.24 (D9)
- net GPIO17: now also A101.23 (D8)
- net GPIO2: now also A101.18 (D3)
- net GPIO25: now also A101.9 (A0)
- net GPIO26: now also A101.10 (A1)
- net GPIO27: now also A101.11 (A2)
- net GPIO32: now also A101.12 (A3)
- net GPIO33: now also A101.13 (SDA/A4)
- net GPIO4: now also A101.19 (D4)
- net IO0: now also A101.17 (D2), R113.2
- net M1_IN1: now also U106.29 (PC6)
- net M1_IN2: now also U106.46 (PB8)
- net M2_IN1: now also U106.47 (PB9)
- net M2_IN2: now also U106.2 (PC13)
- net S0: now also U106.8 (PA0)
- net S1: now also U106.9 (PA1)
- net S2: now also U106.22 (PB10)
- net S3: now also U106.24 (PB11)
- net S4: now also U106.14 (PA6)
- net S5: now also U106.15 (PA7)
- net S6: now also U106.17 (PB0)
- net S7: now also U106.18 (PB1)
- net SCL: now also U106.38 (PA15)
- net SDA: now also U106.45 (PB7)
- net SWCLK: now also U106.37 (PA14), J301.4 (SWCLK)
- net SWDIO: now also U106.36 (PA13), J301.2 (SWDIO)
- net USB_DN: now also U1.4 (IO3), U106.33 (PA11); no longer U1.6 (IO4)
- net USB_DP: now also U1.6 (IO4), U106.34 (PA12); no longer U1.4 (IO3)
- net VREF+: now reaches U106.20 (VREF+)
- net VREF+: now also C126.1, C127.1
- net VBUS/11: now reaches U106.28 (PB15)
- net SWO: now reaches U106.41 (PB3)
- net SWO: now also J301.6 (SWO)
- net BATT/11: now reaches U106.5 (PF0)
- net NRST: now reaches U106.7 (PG10)
- net NRST: now also J301.3 (~{RESET})
- new net RP_PMOS_G: D104.2 (A), Q101.3 (G), R108.1
- new net STM32_EN: R114.1
- new net STM32_IO0: R113.1, S301.2 (NO_2)
- new net VIN: J110.1 (Pin_1), Q101.1 (D_1), Q101.2 (D_2), Q101.5 (D_3), Q101.6 (D_4)
- no-connect marks 11 -> 15
Other:
- note added: "Add more LEDs (maybe a neopixel)"
- note added: "Debug"
- moved on the sheet: C111, C112, C117, U104

Commit message: Firmware working
Parts:
- removed D1: BAT760-115, Diode_SMD:D_SOD-323, symbol Device:D_Schottky
- removed J301: TC2030, Connector:Tag-Connect_TC2030-IDC-FP_2x03_P1.27mm_Vertical, symbol Connector:Conn_ARM_SWD_TagConnect_TC2030
- removed R113: 330R, Resistor_SMD:R_0402_1005Metric, symbol Device:R_Small
- added C2: 22u, Capacitor_SMD:C_0603_1608Metric, symbol Device:C_Small
- added C20: 100n, Capacitor_SMD:C_0402_1005Metric, symbol Device:C_Small
- added D1: LED_R, LED_THT:LED_D5.0mm, symbol Device:LED_Small
- added D2: SK34, 101 Footprints:SK34, symbol SK34-TP:SK34
- added J1: Conn_01x10, 101 Footprints:PinHeader_1x10_P2.54mm_Vertical, symbol Connector_Generic:Conn_01x10
- added J2: Conn_ARM_JTAG_SWD_10, Connector_PinHeader_1.27mm:PinHeader_2x05_P1.27mm_Vertical_SMD, symbol Connector:Conn_ARM_JTAG_SWD_10
- added J3, J4: Conn_01x08, 101 Footprints:PinHeader_1x08_P2.54mm_Vertical, symbol Connector_Generic:Conn_01x08
- added J5: Conn_01x06, 101 Footprints:PinHeader_1x06_P2.54mm_Vertical, symbol Connector_Generic:Conn_01x06
- added R2, R3: 330R, Resistor_SMD:R_0402_1005Metric, symbol Device:R_Small
- added R23: 10k, Resistor_SMD:R_0402_1005Metric, symbol Device:R_Small
- added R4, R5: 2k2, Resistor_SMD:R_0402_1005Metric, symbol Device:R_Small
- A101: footprint 101 Footprints:ICRS_101_UNO_R3 -> 101 Footprints:ICRS_101_UNO_R3_NO_PINS; now not fitted; now left out of the parts list
- C119: footprint Capacitor_SMD:CP_Elec_6.3x5.8 -> Capacitor_THT:CP_Radial_D5.0mm_P2.50mm; now not fitted; now left out of the parts list
- D101, D102: LCSC (none) -> C965804
- D104: LCSC (none) -> C2891751
- IC101, IC103: LCSC (none) -> C1513007
- IC104, IC105: LCSC (none) -> C39159
- J1: footprint 101 Footprints:HRO_TYPE-C-31-M-12 -> MSL Footprints:HRO_TYPE-C-31-M-12; LCSC (none) -> C2765186
- J102, J103, J110: footprint TerminalBlock:TerminalBlock_bornier-2_P5.08mm -> 101 Footprints:TerminalBlock_bornier-2_P5.08mm; now not fitted; now left out of the parts list
- J104, J105, J106, J107, J108, J109: footprint Connector_PinHeader_2.54mm:PinHeader_1x04_P2.54mm_Vertical -> 101 Footprints:PinHeader_1x04_P2.54mm_Vertical; LCSC (none) -> C6332197
- J111: LCSC (none) -> C7430446
- JP401, JP403: footprint Connector_PinHeader_2.54mm:PinHeader_1x03_P2.54mm_Vertical -> 101 Footprints:PinHeader_1x03_P2.54mm_Vertical; LCSC (none) -> C2937625
- L101: footprint Inductor_SMD:L_Chilisin_BMRA00040420 -> 101 Footprints:L_Chilisin_BMRA00040415; LCSC (none) -> C3040385
- L102: footprint Inductor_SMD:L_Chilisin_BMRA00040420 -> 101 Footprints:L_Chilisin_BMRA00040415; LCSC (none) -> C3040384
- Q101: LCSC (none) -> C150441
- R101: value 52k -> 27k
- R102, R105: value 10k -> 5k1
- R103: value 2k2 -> 1k2
- R104: value 31k -> 16k
- R106: value 1k5 -> 330R
- S301: LCSC (none) -> C139797
- U1: LCSC (none) -> C5180279
- U101: footprint RF_Module:ESP32-WROOM-32 -> 101 Footprints:ESP32-WROOM-32; LCSC (none) -> C701342
- U104: LCSC (none) -> C967633
- U106: LCSC (none) -> C529356
Connections:
- net +3.3V: now also J111.2, R23.2, C2.1, J1.3 (Pin_3), J2.1 (VTref), J4.2 (Pin_2), J4.4 (Pin_4), R23.2, R4.2, R5.2
- net +5V: now also JP401.1 (A), JP403.1 (A), J4.5 (Pin_5); no longer C106.1, C107.1, IC103.1 (VIN), IC103.5 (EN), JP401.3 (B), JP403.3 (B)
- net +BATT: now also J110.1 (Pin_1), Q101.1 (D_1), Q101.2 (D_2), Q101.5 (D_3), Q101.6 (D_4), Q101.8 (D_5); no longer A101.8 (VIN), C102.1, C105.1, C114.1, C116.1, C119.1, D104.1 (K), IC101.1 (VIN), IC101.5 (EN), IC104.1 (VM), IC105.1 (VM), Q101.4 (S_1), Q101.7 (S_2), R20.1
- net EN: now also J4.3 (Pin_3)
- net ESP32_RX: now also J3.8 (Pin_8)
- net ESP32_TX: now also J3.7 (Pin_7)
- net GND: now also C2.2, C20.2, J1.4 (Pin_4), J2.3 (GND), J2.5 (GND), J2.9 (GNDDetect), J4.6 (Pin_6), J4.7 (Pin_7), R3.1
- net GPIO12: now also A101.26 (D11), J1.7 (Pin_7); no longer A101.20 (D5)
- net GPIO13: now also A101.28 (D13), J1.5 (Pin_5); no longer A101.21 (D6)
- net GPIO14: now also A101.25 (D10), J1.8 (Pin_8); no longer A101.22 (D7)
- net GPIO15: now also A101.9 (A0), J5.1 (Pin_1); no longer A101.14 (SCL/A5)
- net GPIO16: now also A101.23 (D8), J1.10 (Pin_10); no longer A101.24 (D9)
- net GPIO17: now also A101.22 (D7), J3.1 (Pin_1); no longer A101.23 (D8)
- net GPIO18: now also A101.20 (D5), J3.3 (Pin_3); no longer A101.28 (D13)
- net GPIO19: now also A101.19 (D4), J3.4 (Pin_4); no longer A101.27 (D12)
- net GPIO2: now also A101.27 (D12), J1.6 (Pin_6); no longer A101.18 (D3)
- net GPIO23: now also A101.18 (D3), J3.5 (Pin_5); no longer A101.26 (D11)
- net GPIO25: now also A101.12 (A3), J5.4 (Pin_4); no longer A101.9 (A0)
- net GPIO26: now also A101.11 (A2), J5.3 (Pin_3); no longer A101.10 (A1)
- net GPIO27: now also A101.10 (A1), J5.2 (Pin_2); no longer A101.11 (A2)
- net GPIO32: now also A101.14 (SCL/A5), J5.6 (Pin_6); no longer A101.12 (A3)
- net GPIO33: now also J5.5 (Pin_5)
- net GPIO4: now also A101.24 (D9), J1.9 (Pin_9); no longer A101.19 (D4)
- net GPIO5: now also A101.21 (D6), J3.2 (Pin_2); no longer A101.25 (D10)
- net IO0: now also S301.2 (NO_2), C20.1, J3.6 (Pin_6), R2.2, R23.1
- net M1_IN1: now also U106.8 (PA0); no longer U106.29 (PC6)
- net M1_IN2: now also U106.9 (PA1); no longer U106.46 (PB8)
- net M2_IN2: now also U106.46 (PB8); no longer U106.2 (PC13)
- net MOTOR_SLEEP: now also U106.5 (PF0)
- net NRST: now also J2.10 (~{RESET})
- net S0: now also U106.14 (PA6); no longer U106.8 (PA0)
- net S1: now also U106.15 (PA7); no longer U106.9 (PA1)
- net S2: now also U106.17 (PB0); no longer U106.22 (PB10)
- net S3: now also U106.28 (PB15); no longer U106.24 (PB11)
- net S4: now also U106.29 (PC6); no longer U106.14 (PA6)
- net S5: now also U106.30 (PA8); no longer U106.15 (PA7)
- net S6: now also U106.31 (PA9); no longer U106.17 (PB0)
- net S7: now also U106.32 (PA10); no longer U106.18 (PB1)
- net SCL: now also J1.1 (Pin_1), R5.1
- net SDA: now also J1.2 (Pin_2), R4.1
- net STM32_EN: now also U106.12 (PA4)
- net STM32_IO0: now also U106.13 (PA5), R2.1; no longer S301.2 (NO_2)
- net SWCLK: now also J2.4 (SWDCLK/TCK)
- net SWDIO: now also J2.2 (SWDIO/TMS)
- net SWO: now also J2.6 (SWO/TDO)
- net VBUS: now also D2.2 (A)
- net VBUS/11: now also U106.27 (PB14); no longer U106.28 (PB15)
- net VIN: now also A101.8 (VIN), C102.1, C105.1, C106.1, C107.1, C114.1, C116.1, C119.1, D104.1 (K), IC101.1 (VIN), IC101.5 (EN), IC103.1 (VIN), IC103.5 (EN), IC104.1 (VM), IC105.1 (VM), JP401.3 (B), JP403.3 (B), Q101.4 (S_1), Q101.7 (S_2), R20.1, D2.1 (K), J4.8 (Pin_8); no longer J110.1 (Pin_1), Q101.1 (D_1), Q101.2 (D_2), Q101.5 (D_3), Q101.6 (D_4)
- net VIN/11: now reaches U106.25 (PB12)
- net VIN/11: now also R19.1, R20.2, U101.4 (SENSOR_VP)
- net STM_LED_A: now reaches U106.4 (PC15)
- net STM_LED_A: now also D1.2 (A)
- removed net +3V3: J111.2, JP401.1 (A), JP403.1 (A), R23.2
- removed net BATT/11: R19.1, R20.2, U101.4 (SENSOR_VP), U106.5 (PF0)
- new net STM_LED_K: D1.1 (K), R3.2
- now unconnected: J1.S1 (SHIELD), J1.S2 (SHIELD), J1.S3 (SHIELD), J1.S4 (SHIELD)
- no-connect marks 15 -> 32
Other:
- note added: "I2C PULLUP RESISTORS"
- note removed: "Add more LEDs (maybe a neopixel)"
- moved on the sheet: R114
